File: hw/LCD7Seg.kicad_pcb (KiCad board)
At the start: 2 copper layers, 66 x 45.1 mm, 21 parts, among them J1 Conn_01x07, U1 PCF8562

Commit message: Change i2c address on pcb silkscreen--should be 0x38 and 0x39
Other:
- board text added: "0x38"
- board text added: "0x39"
- board text removed: "0x70"
- board text removed: "0x71"
Changed lines of the file:
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@@
     (effects (font (size 1 1) (thickness 0.2)) (justify mirror))
   )
-  (gr_text 0x71 (at 118.2 75) (layer B.SilkS)
+  (gr_text 0x39 (at 118.2 75) (layer B.SilkS)
     (effects (font (size 1 1) (thickness 0.2)) (justify mirror))
   )
-  (gr_text 0x70 (at 128.2 75) (layer B.SilkS)
+  (gr_text 0x38 (at 128.2 75) (layer B.SilkS)
     (effects (font (size 1 1) (thickness 0.2)) (justify mirror))
   )

Commit message: Migrate to KiCad 7.0
Old files can be found at `legacy/`
KiCad's PCB editor does fills a bit differently now, changing the copper
fill pattern on the board. This warranted a new revision code on the
PCB.
Connections:
- net /~SYNC renamed /~{SYNC}
Other:
- net class Default removed
- board text added: "7Seg LCD Driver 04.2023"
- board text added: "~{SYNC}"
- board text removed: "7Seg LCD Driver 12.2020"
- board text removed: "~SYNC"
